Commit message: URDF changed
Frame of ref shifted along z from COM of Body to between two wheels on their rotational axis.

File: urdf/self_balance_bot.urdf (robot description, URDF)
Before this commit: robot self_balance_bot, 3 links, 2 joints
Links:
- added link body_link, mass 1.00000; collision box size=0.30856 0.40852 0.59953; visual box size=0.30000 0.40000 0.60000
- link base_link: mass 1.00000 -> None; geometry 
Joints:
- added joint body_link_joint: type fixed, parent base_link, child body_link, origin xyz=0.00000 0.00000 0.23648 rpy=0.00000 0.00000 0.00000
- joint wheel_left_link_joint: parent base_link -> body_link
- joint wheel_right_link_joint: parent base_link -> body_link
